Commit message: remove front_left sonar

File: prius_description/urdf/prius.urdf (robot description, URDF)
Before this commit: robot prius, 28 links, 27 joints
Links:
- removed link front_left_far_sonar_link
- removed link front_left_middle_sonar_link
Joints:
- removed joint front_left_far_sonar_joint
- removed joint front_left_middle_sonar_joint
